File: AnalogDiscovery_rs232_5_wire_sniffer.kicad_pcb (KiCad board)
At the start: 2 copper layers, 64 x 64 mm, 23 parts, among them IC1 TCR2EF33,LM_CT, IC2 TRSF3243EIPWR, J1 Conn_02x15_Counter_Clockwise, J2 DE9_Plug, J3 DE9_Receptacle, J4 Conn_02x02_Odd_Even, J5 Conn_02x06_Odd_Even, J6 Conn_02x06_Odd_Even, J7 Conn_02x06_Odd_Even, J8 Conn_02x06_Odd_Even

Commit message: V0.2
Silkscreen changes
Other:
- board text added: "DIO_15: PWR DIO_08: RxD DIO_09: TxD DIO_10: OUT3"
- board text added: "JUBEORMK1 V0.2"
- board text removed: "DIO_15: PWR DIO_08: RxD DIO_09: TxD"
- board text removed: "JUBEORMK1"
Changed lines of the file:
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@@
     (effects (font (size 1 1) (thickness 0.15)) (justify left top mirror))
   )
-  (gr_text "AD ANALOG IN" (at 132.2324 86.4616) (layer "B.SilkS" knockout)
+  (gr_text "AD ANALOG IN" (at 132.2324 88.138) (layer "B.SilkS" knockout)
     (effects (font (size 1 1) (thickness 0.15)) (justify left top mirror))
   )
-  (gr_text "JUBEORMK1" (at 167.2336 127.9856) (layer "B.SilkS")
+  (gr_text "JUBEORMK1 V0.2" (at 167.2336 127.9856) (layer "B.SilkS")
     (effects (font (size 1 1) (thickness 0.15)) (justify left mirror))
   )
-  (gr_text "DIO_15: PWR\nDIO_08: RxD\nDIO_09: TxD" (at 132.2324 80.9752) (layer "B.SilkS")
+  (gr_text "DIO_15: PWR\nDIO_08: RxD\nDIO_09: TxD\nDIO_10: OUT3" (at 132.2324 80.9752) (layer "B.SilkS")
     (effects (font (size 1 1) (thickness 0.15)) (justify left top mirror))
   )
@@
     (effects (font (size 1 1) (thickness 0.15)) (justify left top mirror))
   )
-  (gr_text "SC1_P: RxD\nSC2_P: TxD" (at 132.2324 88.0872) (layer "B.SilkS")
+  (gr_text "SC1_P: RxD\nSC2_P: TxD" (at 132.2324 89.7636) (layer "B.SilkS")
     (effects (font (size 1 1) (thickness 0.15)) (justify left top mirror))
   )
@@
     (effects (font (size 0.8 1) (thickness 0.15)) (justify left top))
   )
-  (gr_text "JUBEORMK1" (at 118.364 127.9144) (layer "F.SilkS")
+  (gr_text "JUBEORMK1 V0.2" (at 118.364 127.9144) (layer "F.SilkS")
     (effects (font (size 1 1) (thickness 0.15)) (justify left))
   )

Commit message: New revision V0.2.1
Small changes:
- Rounded board edges
- better annotation
- C2 is 0603 instead of 0402
- Missing tracks have been removed in J5
Parts:
- C2: footprint Capacitor_SMD:C_0402_1005Metric_Pad0.74x0.62mm_HandSolder -> Capacitor_SMD:C_0603_1608Metric_Pad1.08x0.95mm_HandSolder
- moved C2 1.11 mm to (152.4, 108.4)
Routing:
- net /DTR: track 95.4 -> 93.6 mm
- net /RTS: track 106.8 -> 105.0 mm
- net /RI: track 96.7 -> 95.0 mm
- net /DSR: track 113.3 -> 111.5 mm
- net /DCD: track 114.0 -> 112.2 mm
- net /CTS: track 101.2 -> 99.4 mm
- net +3.3V: track 17.7 -> 19.0 mm
- net GND: track 27.0 -> 28.1 mm
Other:
- outline, holes or cut-outs redrawn
- board text added: "JUBEORMK1 V0.2.1"
- board text added: "SC1_P: RxD (JP1) SC2_P: TxD (JP2)"
- board text removed: "JUBEORMK1 V0.2"
- board text removed: "SC1_P: RxD SC2_P: TxD"
