File: AnalogDiscovery_rs232_5_wire_sniffer.kicad_sch (KiCad schematic)
At the start: 23 parts, among them IC1 TCR2EF33,LM_CT, IC2 TRSF3243EIPWR, J1 Conn_02x15_Counter_Clockwise, J2 DE9_Plug, J3 DE9_Receptacle, J4 Conn_02x02_Odd_Even, J5 Conn_02x06_Odd_Even, J6 Conn_02x06_Odd_Even, J7 Conn_02x06_Odd_Even, J8 Conn_02x06_Odd_Even

Commit message: Added DigiKey part list
Parts:
- J1: Arrow Part Number (none) -> RS:765-5783
- J2: Arrow Part Number (none) -> AE11063-ND
- J3: Arrow Part Number (none) -> AE10972-ND
- J4: Arrow Part Number (none) -> 4324-PHDD-SS004G1ABOGE-B005CT-ND
- J5, J6, J7, J8: Arrow Part Number (none) -> 4324-PHDD-SS016G1ABOGE-B005CT-ND

Commit message: New revision V0.2.1
Small changes:
- Rounded board edges
- better annotation
- C2 is 0603 instead of 0402
- Missing tracks have been removed in J5
Parts:
- C2: footprint Capacitor_SMD:C_0402_1005Metric_Pad0.74x0.62mm_HandSolder -> Capacitor_SMD:C_0603_1608Metric_Pad1.08x0.95mm_HandSolder
Changed lines of the file:
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@@
     (title "Analog Discovery rs232 5 wire sniffer")
     (date "2023-09-29")
-    (rev "V0.1")
+    (rev "V0.2.1")
     (company "JUBEORMK1 @ GITHUB")
+    (comment 1 "Chages: C2 from 0402 to 0603")
   )
